Commit message: initial commit

File: robotiq_2f_140_gripper_visualization/urdf/robotiq_arg2f.xacro (robot description, xacro)
@@ -1,5 +1,5 @@
 <?xml version="1.0"?>
-<robot xmlns:xacro="http://ros.org/wiki/xacro">
-  <xacro:macro name="robotiq_arg2f_base_link" params="prefix">
+<robot name="robotiq_arg2f_140_model" xmlns:xacro="http://ros.org/wiki/xacro">
+  <xacro:macro name="robotiq_arg2f_base_link" params="prefix parent">
     <link name="${prefix}robotiq_arg2f_base_link">
       <inertial>
@@ -24,4 +24,9 @@
       </collision>
     </link>
+    <joint name="tool0-robotiq_arg2f_base_link" type="fixed">
+      <parent link="${parent}"/>
+      <child link="robotiq_arg2f_base_link"/>
+      <origin xyz="0 0 0" rpy="0 0 1.57"/>
+    </joint>
   </xacro:macro>
   <xacro:macro name="finger_joints" params="prefix fingerprefix reflect">

File: robotiq_2f_140_gripper_visualization/urdf/robotiq_arg2f_140_model.xacro (robot description, xacro)
@@ -1,5 +1,6 @@
 <?xml version="1.0"?>
 <robot name="robotiq_arg2f_140_model" xmlns:xacro="http://ros.org/wiki/xacro">
-  <xacro:include filename="$(find robotiq_2f_140_gripper_visualization)/urdf/robotiq_arg2f_140_model_macro.xacro" />
-  <xacro:robotiq_arg2f_140 prefix=""/>
+  <xacro:include filename="$(find robotiq_2f_140_gripper_visualization)/urdf/robotiq_arg2f_140_model_macro.urdf.xacro" />
+  <xacro:robotiq_arg2f_140 prefix="" parent="tool0">
+  </xacro:robotiq_arg2f_140>
 </robot>
